Commit message: Wheels direction has been corrected

File: src/mjf_bunker2_description/src/description/bunker.urdf (robot description, URDF)
Before this commit: robot mjf_bunker2_description, 6 links, 5 joints
Joints:
- removed joint Body_joint
- added joint Robot_Body: type fixed, parent base_link, child Robot_Body, origin xyz=0.0 0.0 0.358 rpy=0.0 0.0 0.0

Commit message: camera and lidar moved _ stable release

File: src/mjf_bunker2_description/src/description/bunker.urdf (robot description, URDF)
Before this commit: robot mjf_bunker2_description, 6 links, 5 joints
Joints:
- joint camera_depth_joint: origin xyz=0.0 0.0 0.0 rpy=${-pi/2} 0 ${-pi/2} -> xyz=0.0 0.0 0.1 rpy=${-pi/2} 0 ${-pi/2}
- joint camera_joint: origin xyz=0.215 0 0.05 rpy=0.0 0.0 0.0 -> xyz=0.215 0 0.15 rpy=0.0 0.0 0.0
- joint lidar_joint: origin xyz=0 0 0.12 rpy=0.0 0.0 0.0 -> xyz=0 0 0.52 rpy=0.0 0.0 0.0
